File: motor-driver.kicad_pcb (KiCad board)
At the start: 4 copper layers, 35 x 27 mm, 112 parts, among them J2 SIGNAL, J3 PWR, J4 RTMI, Q1 BSS138, Q4 SIZ342ADT, Q5 SIZ342ADT, Q6 SIZ342ADT, U1 TMC4671, U2 74LVC3G17, U3 74LVC3G17, U4 TMC6200

Commit message: Optimize the BOM.
Parts:
- C1, C2, C3: value 1nF, 100V -> 1nF
- C10: value 470nF, 50V -> 470nF
- C11, C12, C13, C14, C15, C16, C18, C19, C20, C21, C22, C23, C27, C28, C32, C33, C35, C36, C40, C7, C8: value 100nF, 50V -> 100nF
- C17, C9: value 4.7uF, 16V -> 4.7uF
- C24, C25, C37, C38, C39: value 2.2uF, 50V -> 2.2uF
- C26: value 22nF, 50V -> 22nF
- C29, C30, C31: value 470nF, 16V -> 470nF
- C34: value 47uF, 35V -> 47uF
- C4, C41, C42, C43, C44, C45, C5, C6: value 100pF, 50V -> 100pF
- D1: value 1.6(L)X0.8(W)X0.5(H) MM RED/BLUE -> B2972USNB05
- R1, R10, R11, R12, R15, R16, R2, R20, R21, R22, R23, R3, R4, R5, R6: value 4.7K, %1 -> 4.7K
- R13, TH1: value 10K, %1 -> 10K
- R18: value 47K, %1 -> 47K
- R19, R7, R8, R9: value 1K, %1 -> 1K
- R24, R27, R28, R29, R45: value 270, %1 -> 270
- R25, R26, R46: value 150, %1 -> 150
- R30, R31, R32, R33, R34, R35, R42, R43, R44: value 10, %1 -> 10
- R36, R37, R38, R39, R40, R41: value 0.005, %1, 1W -> 0.005, 1W
